Commit message: debug

File: src/my_robot/urdf/my_robot.xacro (robot description, xacro)
@@ -22,5 +22,5 @@
       <origin xyz="0 0 0" rpy=" 0 0 0"/>
       <geometry>
-        <box size=".4 .2 .1"/>
+        <box size=".4 .1 .1"/>
       </geometry>
     </collision>
@@ -28,5 +28,5 @@
       <origin xyz="0 0 0" rpy=" 0 0 0"/>
       <geometry>
-        <box size=".4 .2 .1"/>
+        <box size=".4 .1 .1"/>
       </geometry>
     </visual>
@@ -80,5 +80,5 @@
  </link>
   <joint type="continuous" name="left_wheel_hinge">
-    <origin xyz="0 0.15 0" rpy="0 0 0"/>
+    <origin xyz="0 0.1 0" rpy="0 0 0"/>
     <child link="left_wheel"/>
     <parent link="chassis"/>
@@ -111,5 +111,5 @@
  </link>
   <joint type="continuous" name="right_wheel_hinge">
-    <origin xyz="0 -0.15 0" rpy="0 0 0"/>
+    <origin xyz="0 -0.1 0" rpy="0 0 0"/>
     <child link="right_wheel"/>
     <parent link="chassis"/>
@@ -177,14 +177,14 @@
   </joint>
  <gazebo reference="left_wheel">
-   <material>Gazebo/Green</material>
+   <material>Gazebo/Yellow</material>
  </gazebo>
  <gazebo reference="right_wheel">
-   <material>Gazebo/Green</material>
+   <material>Gazebo/Yellow</material>
  </gazebo>
  <gazebo reference="chassis">
-   <material>Gazebo/Blue</material>
+   <material>Gazebo/Purple</material>
  </gazebo>
  <gazebo reference="camera">
-   <material>Gazebo/Red</material>
+   <material>Gazebo/Turquoise</material>
  </gazebo>
 </robot>
